File: halflifepcb22.kicad_pcb (KiCad board)
At the start: 2 copper layers, 145 x 105 mm, 27 parts, among them J1 Conn_01x04_Pin, J2 Conn_01x08_Pin, SW1 SW_Push, SW2 SW_Push, U1 XIAO-ESP32-C3-SMD, U2 DHT11

Commit message: Add files via upload
Parts:
- removed the G*** at (213.6, 87.6)
- moved U1 10.7 mm to (204.4, 76.1), turned to 0 degrees
Routing:
- net /SCL: track 400.9 -> 143.7 mm
- net GND: track 49.8 -> 229.3 mm
- net /DHT11 DATA: track 246.2 -> 115.0 mm
- net (no net): track 66.5 -> 3.93 mm
- net +3.3V: track 230.1 -> 174.4 mm
- net /GPIO2: track 123.6 -> 106.7 mm
- net /SDA: track 137.6 -> 153.7 mm
- net /GPIO3: track 46.1 -> 32.5 mm
Other:
- board size 145 x 105 mm -> 140 x 105 mm
